Commit message: OKie dokie

File: src/our_launch/urdf/turtlebot3_waffle_stereo.urdf.xacro (robot description, xacro)
@@ -216,5 +216,5 @@
   <link name="camera_depth_optical_frame"/>
   <joint name="temp" type="fixed">
-    <origin xyz="0 0 0" rpy="-1.57 0 0"/>
+    <origin xyz="0 0 0" rpy="-1.57 0 -1.57"/>
     <parent link="camera_rgb_frame"/>
     <child link="left"/>
